File: GESC_Logic/GESC_Logic-backups/GESC_Logic-2024-12-11_024305/Drivers.kicad_sch (KiCad schematic)
At the start: 27 parts, among them J3 gates_A, J4 gates_B, J5 gates_C, U4 INA240A1D, U5 INA240A1D, U6 INA240A1D, U7 L6498DTR, U8 L6498DTR, U9 L6498DTR

Commit message: update
Parts:
- C15: value 100nF -> 100n
- C16, C17: value 100nF -> 100n; LCSC C14663 -> C14663
- U7, U8, U9: footprint Package_SO:SOIC-8_3.9x4.9mm_P1.27mm -> lcsc:SOIC-8_L4.9-W3.9-P1.27-LS6.0-BL
Changed lines of the file:
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@@
 			)
 		)
-		(property "Value" "100nF"
+		(property "Value" "100n"
 			(at 124.46 40.6462 0)
 			(effects
@@
 			)
 		)
-		(property "Value" "100nF"
+		(property "Value" "100n"
 			(at 124.46 87.6362 0)
 			(effects
@@
 			)
 		)
-		(property "LCSC" "C14663"
+		(property "LCSC" " C14663"
 			(at 121.92 86.36 0)
 			(effects
@@
 			)
 		)
-		(property "Footprint" "Package_SO:SOIC-8_3.9x4.9mm_P1.27mm"
+		(property "Footprint" "lcsc:SOIC-8_L4.9-W3.9-P1.27-LS6.0-BL"
 			(at 128.27 96.52 0)
 			(effects
@@
 			)
 		)
-		(property "Footprint" "Package_SO:SOIC-8_3.9x4.9mm_P1.27mm"
+		(property "Footprint" "lcsc:SOIC-8_L4.9-W3.9-P1.27-LS6.0-BL"
 			(at 128.27 146.05 0)
 			(effects
@@
 			)
 		)
-		(property "Footprint" "Package_SO:SOIC-8_3.9x4.9mm_P1.27mm"
+		(property "Footprint" "lcsc:SOIC-8_L4.9-W3.9-P1.27-LS6.0-BL"
 			(at 128.27 48.26 0)
 			(effects
@@
 			)
 		)
-		(property "Value" "100nF"
+		(property "Value" "100n"
 			(at 124.46 137.1662 0)
 			(effects
@@
 			)
 		)
-		(property "LCSC" "C14663"
+		(property "LCSC" " C14663"
 			(at 121.92 135.89 0)
 			(effects
