File: GESC_Logic/GESC_Logic-backups/GESC_Logic-2024-12-11_024305/GESC_Logic.kicad_pcb (KiCad board)
At the start: 4 copper layers, 100 x 70 mm, 167 parts, among them J1 POWER, J10 DASH/BLE, J11 STLINK, J12 PPM, J13 TYPE-C-31-M-12, J14 BOOT0, J15 NRST, J16 SH1, J17 SH1, J18 SH1, J2 CAN, J3 gates_A, J4 gates_B, J5 gates_C, J6 BMI160, J7 TEMP, J8 BMS, J9 HALL, Q1 BSC320N20NS3G, Q3 BSC320N20NS3G, U1 XL1509-5.0, U10 STM32F405RGTx, U11 LM5146RGYR, U2 LM1117DT-3.3, U3 SN65HVD230DR, U4 INA240A1D, U5 INA240A1D, U6 INA240A1D, U7 L6498DTR, U8 L6498DTR, U9 L6498DTR, Y1 8MHz

Commit message: update
Parts:
- C15, C16, C17: value 100nF -> 100n
- J16, J17, J18: footprint Connector_PinSocket_2.00mm:PinSocket_1x02_P2.00mm_Vertical_SMD_Pin1Left -> Connector_PinSocket_2.00mm:PinSocket_2x01_P2.00mm_Vertical_SMD
- U7, U8, U9: footprint Package_SO:SOIC-8_3.9x4.9mm_P1.27mm -> lcsc:SOIC-8_L4.9-W3.9-P1.27-LS6.0-BL
- moved R29 0.50 mm to (142.2, 102.5)
- moved C30 0.45 mm to (143.5, 104.4), turned to -135 degrees
- turned J16 to 90 degrees
- turned J17 to 90 degrees
- turned J18 to 90 degrees
- turned U7 to -90 degrees
- turned U8 to -90 degrees
- turned U9 to -90 degrees
Connections:
- J14 pad 1: +3V3 -> GND
- R26 pad 1: GND -> +3V3
Routing:
- net +3V3: track 321.5 -> 312.4 mm
- net Net-(C8-Pad1): track 7.14 -> 1.41 mm, vias 2 -> 0
- net SHC_+: track 8.87 -> 9.93 mm
- net GND: track 121.1 -> 120.2 mm
- net SHC_-: track 7.83 -> 8.49 mm
- net SHB_-: track 4.81 -> 5.43 mm
- net SHB_+: track 4.81 -> 5.33 mm
- net SHA_+: track 4.81 -> 5.33 mm
