File: GESC_Logic/GESC_Logic-backups/GESC_Logic-2024-12-11_024305/Logic.kicad_sch (KiCad schematic)
At the start: 78 parts, among them J10 DASH/BLE, J11 STLINK, J12 PPM, J13 TYPE-C-31-M-12, J14 BOOT0, J15 NRST, J6 BMI160, J7 TEMP, J8 BMS, J9 HALL, U10 STM32F405RGTx, Y1 8MHz

Commit message: update
Parts:
- C22, C40: LCSC C14663 -> C14663
- C38: LCSC C14663 -> C60474
- J13: footprint TYPE-C-31-M-12:HRO_TYPE-C-31-M-12 -> Connector_USB:USB_C_Receptacle_HRO_TYPE-C-31-M-12
Connections:
- net +3V3: now also R26.1; no longer J14.1 (Pin_1)
- net GND: now also J14.1 (Pin_1); no longer R26.1
