File: GESC_Logic/GESC_Logic-backups/GESC_Logic-2024-12-11_024305/regulators.kicad_sch (KiCad schematic)
At the start: 48 parts, among them J1 POWER, Q1 BSC320N20NS3G, Q3 BSC320N20NS3G, U1 XL1509-5.0, U11 LM5146RGYR, U2 LM1117DT-3.3

Commit message: update
Parts:
- C5: LCSC C14663 -> C1952781
- L1: LCSC C5298321 -> C5349638
- U1: LCSC C61063 -> C61063
Changed lines of the file:
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@@
 			)
 		)
-		(property "LCSC" "C5298321"
+		(property "LCSC" "C5349638"
 			(at 167.64 43.18 0)
 			(effects
@@
 			)
 		)
-		(property "LCSC" "C14663"
+		(property "LCSC" "C1952781"
 			(at 187.96 91.44 0)
 			(effects
@@
 			)
 		)
-		(property "LCSC" "C61063"
+		(property "LCSC" " C61063"
 			(at 58.42 81.28 0)
 			(effects
