File: GESC_Logic/GESC_Logic.kicad_pcb (KiCad board)
At the start: 4 copper layers, 100 x 64.6 mm, 163 parts, among them J1 POWER, J10 DASH/BLE, J11 STLINK, J12 PPM, J13 TYPE-C-31-M-12, J15 NRST, J16 SH1, J17 SH1, J18 SH1, J2 CAN, J3 gates_A, J4 gates_B, J5 gates_C, J6 BMI160, J7 TEMP, J8 BMS, J9 HALL, Q1 BSC320N20NS3G, Q3 BSC320N20NS3G, U1 XL1509-5.0, U10 STM32F405RGTx, U11 LM5146RGYR, U2 LM1117DT-3.3, U3 SN65HVD230DR, U4 INA241, U5 INA241, U6 INA241, U7 L6498DTR, U8 L6498DTR, U9 L6498DTR, Y1 8MHz

Commit message: asdf
Parts:
- moved F3 4.03 mm to (195.5, 117.0), turned to 180 degrees
- moved C43 0.70 mm to (188.0, 116.8)
- moved R36 0.70 mm to (190.5, 117.5)
- moved R37 0.70 mm to (188.0, 118.4)
Routing:
- net GND: track 116.9 -> 123.6 mm, vias 231 -> 229
- net Net-(J8-Pin_4): track 2.82 -> 5.12 mm
- net +5V: track 177.5 -> 179.8 mm
- net CURRENT_A: track 52.4 -> 54.4 mm
- net Phase_C: track 17.3 -> 15.4 mm
- net V_C: track 45.3 -> 45.9 mm
