File: GESC_Logic/GESC_Logic.kicad_pcb (KiCad board)
At the start: 4 copper layers, 100 x 70 mm, 167 parts, among them J1 POWER, J10 DASH/BLE, J11 STLINK, J12 PPM, J13 TYPE-C-31-M-12, J14 BOOT0, J15 NRST, J16 SH1, J17 SH1, J18 SH1, J2 CAN, J3 gates_A, J4 gates_B, J5 gates_C, J6 BMI160, J7 TEMP, J8 BMS, J9 HALL, Q1 BSC320N20NS3G, Q3 BSC320N20NS3G, U1 XL1509-5.0, U10 STM32F405RGTx, U11 LM5146RGYR, U2 LM1117DT-3.3, U3 SN65HVD230DR, U4 INA240A1D, U5 INA240A1D, U6 INA240A1D, U7 L6498DTR, U8 L6498DTR, U9 L6498DTR, Y1 8MHz

Commit message: asdf
Parts:
- removed C56: 220pF, Capacitor_SMD:C_0402_1005Metric
- removed R45: 59R, Resistor_SMD:R_0805_2012Metric
- U4, U5, U6: value INA240A1D -> INA241; footprint Package_SO:SOIC-8_3.9x4.9mm_P1.27mm -> Package_TO_SOT_SMD:SOT-23-8
- moved C9 3.10 mm to (161.9, 146.6)
- moved C11 2.55 mm to (123.5, 146.5)
- moved C10 2.30 mm to (195.6, 146.4)
- moved U5 1.53 mm to (159.5, 146.6)
- moved U4 1.05 mm to (121.0, 146.6)
- renumbered J14 to BOOT0
Connections:
- C52 pad 1: Net-(U11-EN/UVLO) -> Net-(J1-Pin_1)
- J1 pad 1: +BATT -> Net-(J1-Pin_1)
- R40 pad 1: Net-(U11-EN/UVLO) -> Net-(J1-Pin_1)
- R41 pad 1: Net-(J1-Pin_2) -> +BATT
- R41 pad 2: Net-(U11-EN/UVLO) -> Net-(J1-Pin_1)
- U11 pad 1: Net-(U11-EN/UVLO) -> Net-(J1-Pin_2)
- U11 pad 11: Net-(U11-ILIM) -> unconnected-(U11-ILIM-Pad11)
Routing:
- net Net-(J1-Pin_1): track 0.00 -> 39.7 mm, vias 0 -> 2
- net +3V3: track 321.5 -> 311.8 mm, vias 29 -> 28
- net +BATT: track 134.1 -> 142.4 mm, vias 4 -> 6
- net GND: track 121.1 -> 113.0 mm, vias 254 -> 250
- net Net-(U11-EN/UVLO): track 5.06 -> 0.00 mm
- net SHC_-: track 7.83 -> 3.92 mm
- net Net-(J1-Pin_2): track 42.7 -> 39.7 mm, vias 3 -> 2
- net CURRENT_A: track 53.1 -> 55.6 mm
- net Net-(U11-ILIM): track 2.42 -> 0.00 mm
- net SHC_+: track 8.87 -> 7.21 mm
- net SHB_+: track 4.81 -> 3.60 mm
- net SHB_-: track 4.81 -> 3.66 mm
- net CURRENT_C: track 82.6 -> 83.6 mm
- net SHA_+: track 4.81 -> 4.09 mm
- net SHA_-: track 4.81 -> 4.13 mm
Other:
- board text added: "GND SWC"
- board text added: "SWD 3v3"
- board text added: "{dblquote}Godspeed, braking is for wusses{dblquote}"
- board text removed: "{dblquote}Godspeed, breaking is for wusses{dblquote}"
