File: GESC_Logic/GESC_Logic.kicad_pcb (KiCad board)
At the start: 4 copper layers, 100 x 64.6 mm, 163 parts, among them J1 POWER, J10 DASH/BLE, J11 STLINK, J12 PPM, J13 TYPE-C-31-M-12, J15 NRST, J16 SH1, J17 SH1, J18 SH1, J2 CAN, J3 gates_A, J4 gates_B, J5 gates_C, J6 BMI160, J7 TEMP, J8 BMS, J9 HALL, Q1 BSC320N20NS3G, Q3 BSC320N20NS3G, U1 XL1509-5.0, U10 STM32F405RGTx, U11 LM5146RGYR, U2 LM1117DT-3.3, U3 SN65HVD230DR, U4 INA241, U5 INA241, U6 INA241, U7 L6498DTR, U8 L6498DTR, U9 L6498DTR, Y1 8MHz

Commit message: fffinal
Routing:
- net CURRENT_C: track 107.5 -> 76.5 mm
- net CURRENT_B: track 80.4 -> 53.8 mm
- net CURRENT_A: track 54.4 -> 49.5 mm
- net /Gate Drivers/CH: track 51.4 -> 50.0 mm
- net /Gate Drivers/CL: track 48.1 -> 46.9 mm
Other:
- outline, holes or cut-outs redrawn

Commit message: asdf
Parts:
- moved C11 10.5 mm to (134.5, 135.8)
- moved U4 10.5 mm to (132.0, 135.9)
Changed lines of the file:
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@@
 	(footprint "Package_TO_SOT_SMD:SOT-23-8"
 		(layer "F.Cu")
-		(at 133.125 146.3625 90)
+		(at 132 135.9 90)
 		(descr "SOT, 8 Pin (JEDEC MO-178 Var BA https://www.jedec.org/document_search?search_api_views_fulltext=MO-178), generated with kicad-footprint-generator ipc_gullwing_generator.py")
 		(tags "SOT TO_SOT_SMD")
@@
 	(footprint "Capacitor_SMD:C_0603_1608Metric"
 		(layer "F.Cu")
-		(at 135.625 146.3125 -90)
+		(at 134.5 135.85 -90)
 		(descr "Capacitor SMD 0603 (1608 Metric), square (rectangular) end terminal, IPC_7351 nominal, (Body size source: IPC-SM-782 page 76, https://www.pcb-3d.com/wordpress/wp-content/uploads/ipc-sm-782a_amendment_1_and_2.pdf), generated with kicad-footprint-generator")
 		(tags "capacitor")
@@
 	)
 	(segment
-		(start 134.1 147.5)
-		(end 132.85 147.5)
+		(start 132.975 137.0375)
+		(end 131.725 137.0375)
 		(width 0.5)
 		(layer "F.Cu")
@@
 	)
 	(segment
-		(start 135.625 147.0875)
-		(end 134.5125 147.0875)
+		(start 134.5 136.625)
+		(end 133.3875 136.625)
 		(width 0.5)
 		(layer "F.Cu")
@@
 	)
 	(segment
-		(start 134.5125 147.0875)
-		(end 134.1 147.5)
+		(start 133.3875 136.625)
+		(end 132.975 137.0375)
 		(width 0.5)
 		(layer "F.Cu")
@@
 	)
 	(via
-		(at 135.625 148.1125)
+		(at 134.5 137.65)
 		(size 0.6)
 		(drill 0.3)
@@
 	)
 	(via
-		(at 136.725 147.0125)
+		(at 135.6 136.55)
 		(size 0.6)
 		(drill 0.3)
@@
 	)
 	(segment
-		(start 132.85 145.454138)
-		(end 132.85 145.225)
+		(start 131.725 134.991638)
+		(end 131.725 134.7625)
 		(width 0.5)
 		(layer "F.Cu")
@@
 	)
 	(segment
-		(start 134.8 146.3625)
-		(end 134.075 146.3625)
+		(start 133.675 135.9)
+		(end 132.95 135.9)
 		(width 0.5)
 		(layer "F.Cu")
@@
 	)
 	(segment
-		(start 134.075 146.3625)
-		(end 133.758362 146.3625)
+		(start 132.95 135.9)
+		(end 132.633362 135.9)
 		(width 0.5)
 		(layer "F.Cu")
@@
 	)
 	(segment
-		(start 135.625 145.5375)
-		(end 135.0625 146.1)
+		(start 134.5 135.075)
+		(end 133.9375 135.6375)
 		(width 0.5)
 		(layer "F.Cu")
@@
 	)
 	(segment
-		(start 133.758362 146.3625)
-		(end 133.141681 145.745819)
+		(start 132.633362 135.9)
+		(end 132.016681 135.283319)
 		(width 0.5)
 		(layer "F.Cu")
@@
 	)
 	(segment
-		(start 135.0625 146.1)
-		(end 134.8 146.3625)
+		(start 133.9375 135.6375)
+		(end 133.675 135.9)
 		(width 0.5)
 		(layer "F.Cu")
@@
 	)
 	(segment
-		(start 133.141681 145.745819)
-		(end 132.85 145.454138)
+		(start 132.016681 135.283319)
+		(end 131.725 134.991638)
 		(width 0.5)
 		(layer "F.Cu")
@@
 	)
 	(via
-		(at 133.141681 145.745819)
+		(at 132.016681 135.283319)
 		(size 0.6)
 		(drill 0.3)
@@
 	)
 	(via
-		(at 135.0625 146.1)
+		(at 133.9375 135.6375)
 		(size 0.6)
 		(drill 0.3)
@@
 	)
 	(segment
-		(start 135.766681 145.745819)
-		(end 133.141681 145.745819)
+		(start 134.641681 135.283319)
+		(end 132.016681 135.283319)
 		(width 1)
 		(layer "B.Cu")
@@
 	)
 	(segment
-		(start 136.1 145.4125)
-		(end 135.766681 145.745819)
+		(start 134.975 134.95)
+		(end 134.641681 135.283319)
 		(width 1)
 		(layer "B.Cu")
@@
 	)
 	(segment
-		(start 132.1 147.45)
-		(end 132.1 147.5)
+		(start 130.975 136.9875)
+		(end 130.975 137.0375)
 		(width 0.5)
 		(layer "F.Cu")
@@
 	)
 	(segment
-		(start 129.675 147.4125)
-		(end 132.0625 147.4125)
+		(start 128.55 136.95)
+		(end 130.9375 136.95)
 		(width 0.5)
 		(layer "F.Cu")
@@
 	)
 	(segment
-		(start 132.0625 147.4125)
-		(end 132.1 147.45)
+		(start 130.9375 136.95)
+		(end 130.975 136.9875)
 		(width 0.5)
 		(layer "F.Cu")
@@
 	)
 	(via
-		(at 129.675 147.4125)
+		(at 128.55 136.95)
 		(size 0.6)
 		(drill 0.3)
@@
 	)
 	(segment
-		(start 132.1 145.275)
-		(end 132.1 145.225)
+		(start 130.975 134.8125)
+		(end 130.975 134.7625)
 		(width 0.5)
 		(layer "F.Cu")
@@
 	)
 	(segment
-		(start 131.275 145.3125)
-		(end 132.0625 145.3125)
+		(start 130.15 134.85)
+		(end 130.9375 134.85)
 		(width 0.5)
 		(layer "F.Cu")
@@
 	)
 	(segment
-		(start 132.0625 145.3125)
-		(end 132.1 145.275)
+		(start 130.9375 134.85)
+		(end 130.975 134.8125)
 		(width 0.5)
 		(layer "F.Cu")
@@
 	)
 	(via
-		(at 131.275 145.3125)
+		(at 130.15 134.85)
 		(size 0.6)
 		(drill 0.3)
@@
 	)
 	(segment
-		(start 130.1625 145.3125)
-		(end 129.95 145.1)
+		(start 129.0375 134.85)
+		(end 128.825 134.6375)
 		(width 0.5)
 		(layer "B.Cu")
@@
 	)
 	(segment
-		(start 131.275 145.3125)
-		(end 130.1625 145.3125)
+		(start 130.15 134.85)
+		(end 129.0375 134.85)
 		(width 0.5)
 		(layer "B.Cu")

Commit message: 1
Routing:
- net CURRENT_A: track 49.5 -> 38.5 mm
- net SHA_+: track 2.30 -> 11.2 mm
- net SHA_-: track 6.96 -> 13.8 mm
- net +3V3: track 296.5 -> 298.4 mm
Changed lines of the file:
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@@
 	)
 	(segment
+		(start 134.026 135.549)
+		(end 133.9375 135.6375)
+		(width 1)
+		(layer "B.Cu")
+		(net 3)
+	)
+	(segment
 		(start 159.7 140.6)
 		(end 162 140.6)
@@
 	)
 	(segment
+		(start 136.014628 135.549)
+		(end 134.026 135.549)
+		(width 1)
+		(layer "B.Cu")
+		(net 3)
+	)
+	(segment
+		(start 140.9125 140.446872)
+		(end 136.014628 135.549)
+		(width 1)
+		(layer "B.Cu")
+		(net 3)
+	)
+	(segment
 		(start 162 140.6)
 		(end 186.1 140.6)
@@
 	)
 	(segment
-		(start 140.9125 140.6)
-		(end 136.1 145.4125)
-		(width 1)
-		(layer "B.Cu")
-		(net 3)
-	)
-	(segment
 		(start 188.145 93.2)
 		(end 189.6 91.745)
@@
 	)
 	(segment
-		(start 134.975 134.95)
-		(end 134.641681 135.283319)
+		(start 140.9125 140.6)
+		(end 140.9125 140.446872)
 		(width 1)
 		(layer "B.Cu")
@@
 	)
 	(segment
-		(start 143.25 111.8)
-		(end 143.25 111.190559)
-		(width 0.2)
-		(layer "F.Cu")
-		(net 7)
-	)
-	(segment
-		(start 146.498097 107.648349)
-		(end 146.498097 107.942462)
+		(start 140.651304 111.975)
+		(end 140.35 112.276304)
 		(width 0.2)
 		(layer "F.Cu")
@@
 	)
 	(segment
-		(start 132.3 131.881372)
-		(end 134.1 133.681372)
+		(start 143.25 111.8)
+		(end 143.25 111.190559)
 		(width 0.2)
 		(layer "F.Cu")
@@
 	)
 	(segment
-		(start 140.35 112.276304)
-		(end 140.35 113.4)
+		(start 146.498097 107.648349)
+		(end 146.498097 107.942462)
 		(width 0.2)
 		(layer "F.Cu")
@@
 	)
 	(segment
-		(start 132.3 118.7)
-		(end 132.3 131.881372)
-		(width 0.2)
-		(layer "F.Cu")
-		(net 7)
-	)
-	(segment
 		(start 143.075 112.325)
 		(end 142.65 112.75)
@@
 	)
 	(segment
-		(start 140.35 113.4)
-		(end 138.15 115.6)
+		(start 135.4 115.6)
+		(end 132.3 118.7)
 		(width 0.2)
 		(layer "F.Cu")
@@
 	)
 	(segment
-		(start 135.4 115.6)
-		(end 132.3 118.7)
+		(start 132.3 118.7)
+		(end 132.3 131.881372)
 		(width 0.2)
 		(layer "F.Cu")
@@
 	)
 	(segment
-		(start 134.1 133.681372)
-		(end 134.1 145.225)
+		(start 132.3 131.881372)
+		(end 132.975 132.556372)
+		(width 0.2)
+		(layer "F.Cu")
+		(net 7)
+	)
+	(segment
+		(start 132.975 132.556372)
+		(end 132.975 134.7625)
 		(width 0.2)
 		(layer "F.Cu")
@@
 	)
 	(segment
-		(start 140.651304 111.975)
-		(end 140.35 112.276304)
+		(start 140.35 112.276304)
+		(end 140.35 113.4)
+		(width 0.2)
+		(layer "F.Cu")
+		(net 7)
+	)
+	(segment
+		(start 140.35 113.4)
+		(end 138.15 115.6)
 		(width 0.2)
 		(layer "F.Cu")
@@
 	)
 	(segment
-		(start 129.675 147.4125)
-		(end 127.0625 147.4125)
-		(width 0.5)
-		(layer "B.Cu")
-		(net 81)
-	)
-	(segment
-		(start 127.8625 147.1)
-		(end 128.075 147.3125)
+		(start 127.0625 147.4125)
+		(end 126.75 147.1)
 		(width 0.5)
 		(layer "B.Cu")
@@
 	)
 	(segment
-		(start 126.75 147.1)
-		(end 127.8625 147.1)
+		(start 128.55 136.95)
+		(end 126.75 138.75)
 		(width 0.5)
 		(layer "B.Cu")
@@
 	)
 	(segment
-		(start 127.0625 147.4125)
+		(start 126.75 138.75)
 		(end 126.75 147.1)
 		(width 0.5)
@@
 	)
 	(segment
-		(start 129.0375 134.85)
-		(end 128.825 134.6375)
+		(start 129.95 135.05)
+		(end 129.95 145.1)
 		(width 0.5)
 		(layer "B.Cu")
@@
 	(segment
 		(start 130.15 134.85)
-		(end 129.0375 134.85)
+		(end 129.95 135.05)
 		(width 0.5)
 		(layer "B.Cu")
