File: GESC_Logic/Logic.kicad_sch (KiCad schematic)
At the start: 78 parts, among them J10 DASH/BLE, J11 STLINK, J12 PPM, J13 TYPE-C-31-M-12, J14 BOOT0, J15 NRST, J6 BMI160, J7 TEMP, J8 BMS, J9 HALL, U10 STM32F405RGTx, Y1 8MHz

Commit message: asdf
Parts:
- R32, R34, R36: value 150k -> 360k
- R33, R35, R37: value 3.3k -> 8.2k
Changed lines of the file:
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@@
 		(shape input)
 		(at 201.93 134.62 0)
-		(fields_autoplaced yes)
 		(effects
 			(font
@@
 		(shape input)
 		(at 201.93 139.7 0)
-		(fields_autoplaced yes)
 		(effects
 			(font
@@
 		(shape input)
 		(at 201.93 83.82 0)
-		(fields_autoplaced yes)
 		(effects
 			(font
@@
 		(shape input)
 		(at 201.93 81.28 0)
-		(fields_autoplaced yes)
 		(effects
 			(font
@@
 		(shape input)
 		(at 228.6 36.83 180)
-		(fields_autoplaced yes)
 		(effects
 			(font
@@
 		(shape input)
 		(at 201.93 137.16 0)
-		(fields_autoplaced yes)
 		(effects
 			(font
@@
 		(shape input)
 		(at 201.93 142.24 0)
-		(fields_autoplaced yes)
 		(effects
 			(font
@@
 		(shape input)
 		(at 201.93 86.36 0)
-		(fields_autoplaced yes)
 		(effects
 			(font
@@
 		(shape input)
 		(at 255.27 20.32 180)
-		(fields_autoplaced yes)
 		(effects
 			(font
@@
 			)
 		)
-		(property "Value" "150k"
+		(property "Value" "360k"
 			(at 252.73 135.89 0)
 			(effects
@@
 			)
 		)
-		(property "Value" "150k"
+		(property "Value" "360k"
 			(at 252.73 102.87 0)
 			(effects
@@
 			)
 		)
-		(property "Value" "3.3k"
+		(property "Value" "8.2k"
 			(at 252.73 147.32 0)
 			(effects
@@
 			)
 		)
-		(property "Value" "3.3k"
+		(property "Value" "8.2k"
 			(at 252.73 114.3 0)
 			(effects
@@
 			)
 		)
-		(property "Value" "3.3k"
+		(property "Value" "8.2k"
 			(at 252.73 81.28 0)
 			(effects
@@
 			)
 		)
-		(property "Value" "150k"
+		(property "Value" "360k"
 			(at 252.73 69.85 0)
 			(effects
