File: GESC_Logic/regulators.kicad_sch (KiCad schematic)
At the start: 48 parts, among them J1 POWER, Q1 BSC320N20NS3G, Q3 BSC320N20NS3G, U1 XL1509-5.0, U11 LM5146RGYR, U2 LM1117DT-3.3

Commit message: asdf
Parts:
- removed C56: 220pF, Capacitor_SMD:C_0402_1005Metric, symbol Device:C_Small
- removed R45: 59R, Resistor_SMD:R_0805_2012Metric, symbol Device:R_Small
Connections:
- net +BATT: now also R41.1; no longer J1.1 (Pin_1)
- net at C52.1, R40.1, R41.2: now also J1.1 (Pin_1); no longer U11.1 (EN/UVLO)
- net at J1.2 (Pin_2): now also U11.1 (EN/UVLO); no longer R41.1
- no-connect marks 1 -> 2
Other:
- moved on the sheet: J1

Commit message: asdf
Other:
- moved on the sheet: C1, C2, C3, C61, C62, C63, D8, L2, U1
